Commit message: feat: Successfully launched tutorial robot in Gazebo

File: robot_arm_urdf/urdf/robot_arm_urdf.urdf (robot description, URDF)
Before this commit: robot robot_arm_urdf, 8 links, 7 joints
Links:
- added link world
Joints:
- added joint base_joint: type fixed, parent world, child base_link, origin xyz=0 0 0.17 rpy=0 0 0
- joint joint_4: limit lower=0 upper=-3.142 effort=200 velocity=3 -> lower=-3.142 upper=0 effort=200 velocity=3

Commit message: feat: Pipeline validation complete - Gazebo and MoveIt working

File: robot_arm_urdf/urdf/robot_arm_urdf.urdf (robot description, URDF)
Before this commit: robot robot_arm_urdf, 9 links, 8 joints
Joints:
- joint joint_1: limit lower=0 upper=3.142 effort=300 velocity=3 -> lower=0 upper=6.284 effort=300 velocity=3
- joint joint_3: limit lower=0 upper=3.142 effort=200 velocity=3 -> lower=-3.142 upper=0 effort=200 velocity=3

Commit message: feat: Add working color detection node and simulated world

File: robot_arm_urdf/urdf/robot_arm_urdf.urdf (robot description, URDF)
Before this commit: robot robot_arm_urdf, 9 links, 8 joints
Links:
- added link camera_link
Joints:
- added joint camera_joint: type fixed, parent base_link, child camera_link, origin xyz=0.4 0.0 0.8 rpy=0 1.57 0

Commit message: Fix: Correct launch files and URDF for stable simulation

File: robot_arm_urdf/urdf/robot_arm_urdf.urdf (robot description, URDF)
Before this commit: robot robot_arm_urdf, 10 links, 9 joints
Joints:
- joint base_joint: origin xyz=0 0 0.17 rpy=0 0 0 -> xyz=0 0 0 rpy=0 0 0
- joint camera_joint: origin xyz=0.4 0.0 0.8 rpy=0 1.57 0 -> xyz=0.0 -0.693 0.8 rpy=0 1.57 0
