Commit message: feat: Complete and calibrate perception-to-control pipeline

File: robot_arm_urdf/urdf/camera.xacro (robot description, xacro)
@@ -2,4 +2,5 @@
 <robot xmlns:xacro="http://www.ros.org/wiki/xacro">
   <xacro:macro name="waste_camera">
+    <link name="world"/>
     <link name="waste_camera_link">
       <visual>
@@ -13,7 +14,7 @@
     </link>
     <joint name="waste_camera_joint" type="fixed">
-      <parent link="base_link"/>
+      <parent link="world"/>
       <child link="waste_camera_link"/>
-      <origin xyz="0.0 -0.693 0.8" rpy="0 1.57 0"/>
+      <origin xyz="0.0 -0.60 0.8" rpy="0 1.5707 0"/>
     </joint>
     <gazebo reference="waste_camera_link">
@@ -35,5 +36,6 @@
           <alwaysOn>true</alwaysOn>
           <updateRate>0.0</updateRate>
-          <cameraName>waste_camera</cameraName> <imageTopicName>image_raw</imageTopicName>
+          <cameraName>waste_camera</cameraName>
+          <imageTopicName>image_raw</imageTopicName>
           <cameraInfoTopicName>camera_info</cameraInfoTopicName>
           <frameName>waste_camera_link</frameName>

File: robot_arm_urdf/urdf/robot_arm_urdf.urdf (robot description, URDF)
Before this commit: robot robot_arm_urdf, 10 links, 9 joints
Joints:
- joint camera_joint: origin xyz=0.0 -0.693 0.8 rpy=0 1.57 0 -> xyz=0.0 -0.60 0.8 rpy=0 1.5707 0
